File: schémata/security_system/security_system.kicad_sch (KiCad schematic)
At the start: 1 part

Commit message: add readme and scheme
Parts:
- removed U?: STM8S003F3P, Package_SO:TSSOP-20_4.4x6.5mm_P0.65mm, symbol MCU_ST_STM8:STM8S003F3P
- added J?: USB_A_{2}, symbol Connector:USB_A
- added J?: USB_A_{1}, symbol Connector:USB_A
- added Programátor, USB/TTL_převodník: ZL201-04G, Connector_PinHeader_2.54mm:PinHeader_1x04_P2.54mm_Vertical, symbol KLIB_Connector_Prog:ST_SWIM_01X04
- added U?: RFID RC-522, MODULE_CEG006900, symbol CEG006900:CEG006900
- added U?: STM8S103F3M6, Package_SO:SO-20_12.8x7.5mm_P1.27mm, symbol KLIB_MCU_ST_STM8S:STM8S103F3M
- added U?: PCF8574, Display:LCD-016N002L, symbol Display_Character:LCD-016N002L
- added U?: LCD1602, Display:LCD-016N002L, symbol Display_Character:LCD-016N002L
Connections:
- new net: U?.1 (V_{CC}), U?.1 (V_{CC})
- new net: U?.10 (DB3), U?.10 (DB3)
- new net: U?.11 (DB4), U?.11 (DB4)
- new net: U?.12 (DB5), U?.12 (DB5)
- new net: U?.13 (DB6), U?.13 (DB6)
- new net: U?.14 (DB7), U?.14 (DB7)
- new net: U?.15 (A/VEE), U?.15 (A/VEE)
- new net: U?.16 (K), U?.16 (K)
- new net: U?.2 (V_{DD}), U?.2 (V_{DD})
- new net: U?.3 (VO), U?.3 (VO)
- new net: U?.4 (RS), U?.4 (SCL)
- new net: U?.5 (R/~{W}), U?.5 (R/~{W})
- new net: U?.6 (E), U?.6 (E)
- new net: U?.7 (DB0), U?.7 (SDA)
- new net: U?.8 (DB1), U?.8 (DB1)
- new net: U?.9 (DB2), U?.9 (DB2)
- new net: U?.A1, U?.A1
- new net: U?.A2, U?.A2
- new net: U?.K1, U?.K1
- new net: U?.K2, U?.K2
- new net GND: Programátor.3 (GND), U?.2 (V_{DD}), U?.3 (GND), U?.7 (V_{SS}), USB/TTL_převodník.2 (GND)
- new net MISO: U?.17 (PC7)
- new net MOSI: U?.16 (PC6)
- new net PB4: U?.4 (SCL)
- new net PB5: U?.7 (SDA)
- new net PC3: U?.2 (RST)
- new net PC4: U?.8 (SS)
- new net PC5: U?.7 (SCK)
- new net PC6: U?.6 (MOSI)
- new net PC7: U?.5 (MISO)
- new net PD1: Programátor.2 (SWIM)
- new net PD5: USB/TTL_převodník.4 (Rx)
- new net PD6: USB/TTL_převodník.3 (Tx)
- new net RST: U?.13 (PC3)
- new net Rx: U?.2 (PD5)
- new net SCK: U?.15 (PC5)
- new net SCL: U?.11 (PB5)
- new net SDA: U?.12 (PB4)
- new net SS: U?.14 (PC4)
- new net SWIM: U?.18 (PD1)
- new net Tx: U?.3 (PD6)
- new net VDD: U?.9 (V_{DD})
- new net V_{CC}: U?.2 (V_{DD})
- new net V_{DD}: U?.1 (V_{CC}), USB/TTL_převodník.1 (V_{CC})
- new net ~{RST}: Programátor.4 (~{RST}), U?.4 (NRST)
Other:
- note added: "DeroBoard"
- note added: "I2C převodník s displejem LCD1602"
- note added: "Programátor"
- note added: "Serial monitor bridge"
- note added: "Čtečka RFID karet"
- title: (none) -> Security system

Commit message: add readme and scheme
Parts:
- added D_{1}: GREEN, symbol Device:LED
- added D_{2}: RED, symbol Device:LED
- added R_{1}, R_{2}: 300R, symbol Device:R
Connections:
- net GND: now also D_{1}.1 (K), D_{2}.1 (K)
- net at U?.5 (PA1): now also R_{1}.2
- net at U?.6 (PA2): now also R_{2}.2
- new net: D_{2}.2 (A), R_{2}.1
- new net: D_{1}.2 (A), R_{1}.1
Changed lines of the file:
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@@
     (rev "Petr Oblouk")
+  )
+  (junction (at 26.67 147.32) (diameter 0) (color 0 0 0 0)
   )
   (bus_entry (at 246.38 52.07) (size 2.54 2.54)
@@
     (stroke (width 0) (type default) (color 0 0 0 0))
   )
+  (wire (pts (xy 46.99 135.89) (xy 52.07 135.89))
+    (stroke (width 0) (type default) (color 0 0 0 0))
+  )
   (wire (pts (xy 102.87 151.13) (xy 115.57 151.13))
+    (stroke (width 0) (type default) (color 0 0 0 0))
+  )
+  (wire (pts (xy 72.39 143.51) (xy 52.07 143.51))
     (stroke (width 0) (type default) (color 0 0 0 0))
   )
@@
     (stroke (width 0) (type default) (color 0 0 0 0))
   )
+  (wire (pts (xy 36.83 147.32) (xy 39.37 147.32))
+    (stroke (width 0) (type default) (color 0 0 0 0))
+  )
   (bus (pts (xy 229.87 88.9) (xy 246.38 88.9))
     (stroke (width 0) (type default) (color 0 0 0 0))
@@
     (stroke (width 0) (type default) (color 0 0 0 0))
   )
+  (wire (pts (xy 26.67 147.32) (xy 29.21 147.32))
+    (stroke (width 0) (type default) (color 0 0 0 0))
+  )
   (wire (pts (xy 120.65 57.15) (xy 133.35 57.15))
     (stroke (width 0) (type default) (color 0 0 0 0))
@@
   )
   (bus (pts (xy 246.38 88.9) (xy 246.38 92.71))
+    (stroke (width 0) (type default) (color 0 0 0 0))
+  )
+  (wire (pts (xy 52.07 140.97) (xy 72.39 140.97))
+    (stroke (width 0) (type default) (color 0 0 0 0))
+  )
+  (wire (pts (xy 29.21 135.89) (xy 26.67 135.89))
     (stroke (width 0) (type default) (color 0 0 0 0))
   )
@@
     (stroke (width 0) (type default) (color 0 0 0 0))
   )
+  (wire (pts (xy 52.07 143.51) (xy 52.07 147.32))
+    (stroke (width 0) (type default) (color 0 0 0 0))
+  )
   (wire (pts (xy 77.47 80.01) (xy 97.79 80.01))
     (stroke (width 0) (type default) (color 0 0 0 0))
@@
     (stroke (width 0) (type solid) (color 0 0 0 0))
   )
+  (wire (pts (xy 52.07 135.89) (xy 52.07 140.97))
+    (stroke (width 0) (type default) (color 0 0 0 0))
+  )
   (wire (pts (xy 207.01 91.44) (xy 194.31 91.44))
+    (stroke (width 0) (type default) (color 0 0 0 0))
+  )
+  (wire (pts (xy 52.07 147.32) (xy 46.99 147.32))
     (stroke (width 0) (type default) (color 0 0 0 0))
   )
@@
     (stroke (width 0) (type default) (color 0 0 0 0))
   )
+  (wire (pts (xy 26.67 147.32) (xy 26.67 151.13))
+    (stroke (width 0) (type default) (color 0 0 0 0))
+  )
   (polyline (pts (xy 176.53 13.97) (xy 176.53 163.83))
     (stroke (width 0) (type default) (color 0 0 0 0))
@@
   )
   (wire (pts (xy 194.31 35.56) (xy 209.55 35.56))
+    (stroke (width 0) (type default) (color 0 0 0 0))
+  )
+  (wire (pts (xy 36.83 135.89) (xy 39.37 135.89))
+    (stroke (width 0) (type default) (color 0 0 0 0))
+  )
+  (wire (pts (xy 26.67 135.89) (xy 26.67 147.32))
     (stroke (width 0) (type default) (color 0 0 0 0))
   )
@@
     (pin "K2")
   )
+  (symbol (lib_id "Device:LED") (at 33.02 147.32 0) (unit 1)
+    (in_bom yes) (on_board yes)
+    (property "Reference" "D_{2}" (id 0) (at 33.02 142.24 0)
+      (effects (font (size 1.27 1.27) bold))
+    )
+    (property "Value" "RED" (id 1) (at 33.02 144.78 0))
+    (property "Footprint" "" (id 2) (at 33.02 147.32 0)
+      (effects (font (size 1.27 1.27)) hide)
+    )
+    (property "Datasheet" "~" (id 3) (at 33.02 147.32 0)
+      (effects (font (size 1.27 1.27)) hide)
+    )
+    (pin "1")
+    (pin "2")
+  )
+  (symbol (lib_id "Device:R") (at 43.18 135.89 90) (unit 1)
+    (in_bom yes) (on_board yes)
+    (property "Reference" "R_{1}" (id 0) (at 45.72 130.81 90)
+      (effects (font (size 1.27 1.27) bold))
+    )
+    (property "Value" "300R" (id 1) (at 46.99 133.35 90))
+    (property "Footprint" "" (id 2) (at 43.18 137.668 90)
+      (effects (font (size 1.27 1.27)) hide)
+    )
+    (property "Datasheet" "~" (id 3) (at 43.18 135.89 0)
+      (effects (font (size 1.27 1.27)) hide)
+    )
+    (pin "1")
+    (pin "2")
+  )
   (symbol (lib_id "KLIB_Connector_Prog:ST_SWIM_01X04") (at 214.63 35.56 0) (mirror y) (unit 1)
     (in_bom yes) (on_board yes)
@@
     )
     (pin "1")
+  )
+  (symbol (lib_id "Device:LED") (at 33.02 135.89 0) (unit 1)
+    (in_bom yes) (on_board yes)
+    (property "Reference" "D_{1}" (id 0) (at 33.02 130.81 0)
+      (effects (font (size 1.27 1.27) bold))
+    )
+    (property "Value" "GREEN" (id 1) (at 34.29 133.35 0))
+    (property "Footprint" "" (id 2) (at 33.02 135.89 0)
+      (effects (font (size 1.27 1.27)) hide)
+    )
+    (property "Datasheet" "~" (id 3) (at 33.02 135.89 0)
+      (effects (font (size 1.27 1.27)) hide)
+    )
+    (pin "1")
+    (pin "2")
   )
   (symbol (lib_id "KLIB_Power:GND") (at 200.66 97.79 0) (unit 1)
@@
     (pin "K2")
   )
+  (symbol (lib_id "Device:R") (at 43.18 147.32 90) (unit 1)
+    (in_bom yes) (on_board yes)
+    (property "Reference" "R_{2}" (id 0) (at 45.72 142.24 90)
+      (effects (font (size 1.27 1.27) bold))
+    )
+    (property "Value" "300R" (id 1) (at 46.99 144.78 90))
+    (property "Footprint" "" (id 2) (at 43.18 149.098 90)
+      (effects (font (size 1.27 1.27)) hide)
+    )
+    (property "Datasheet" "~" (id 3) (at 43.18 147.32 0)
+      (effects (font (size 1.27 1.27)) hide)
+    )
+    (pin "1")
+    (pin "2")
+  )
   (symbol (lib_id "KLIB_Power:GND") (at 125.73 64.77 0) (unit 1)
     (in_bom yes) (on_board yes) (fields_autoplaced)
@@
     (pin "1")
   )
+  (symbol (lib_id "KLIB_Power:GND") (at 26.67 151.13 0) (unit 1)
+    (in_bom yes) (on_board yes) (fields_autoplaced)
+    (property "Reference" "#PWR?" (id 0) (at 26.67 156.21 0)
+      (effects (font (size 1.27 1.27)) hide)
+    )
+    (property "Value" "GND" (id 1) (at 26.67 155.8196 0))
+    (property "Footprint" "" (id 2) (at 26.67 151.13 0)
+      (effects (font (size 1.27 1.27)) hide)
+    )
+    (property "Datasheet" "" (id 3) (at 26.67 151.13 0)
+      (effects (font (size 1.27 1.27)) hide)
+    )
+    (pin "1")
+  )
   (sheet_instances
     (path "/" (page "1"))
@@
       (reference "#PWR?") (unit 1) (value "GND") (footprint "")
     )
+    (path "/fc03d718-1ba4-4473-aada-aca7cdcb06f4"
+      (reference "#PWR?") (unit 1) (value "GND") (footprint "")
+    )
+    (path "/d56ca87e-6ee6-47c6-9e81-7a8d239c9808"
+      (reference "D_{1}") (unit 1) (value "GREEN") (footprint "")
+    )
+    (path "/61fd40f0-d683-462c-b51c-32aa99ad106a"
+      (reference "D_{2}") (unit 1) (value "RED") (footprint "")
+    )
     (path "/98fdf933-9585-4845-95e1-d8aa256b3006"
       (reference "J?") (unit 1) (value "USB_A_{2}") (footprint "")
@@
       (reference "Programátor") (unit 1) (value "ZL201-04G") (footprint "Connector_PinHeader_2.54mm:PinHeader_1x04_P2.54mm_Vertical")
     )
+    (path "/742fd7ac-55f2-4bed-a58d-b7192fe1e1f6"
+      (reference "R_{1}") (unit 1) (value "300R") (footprint "")
+    )
+    (path "/eed3091a-5973-4ce0-a2ac-ff8fc3a25e0a"
+      (reference "R_{2}") (unit 1) (value "300R") (footprint "")
+    )
     (path "/1dfbb7ef-5d23-48f8-8a35-4e185d62750c"

Commit message: update
Parts:
- removed U?: STM8S103F3M6, Package_SO:SO-20_12.8x7.5mm_P1.27mm, symbol KLIB_MCU_ST_STM8S:STM8S103F3M
- added CN1, CN2, CN3, CN4: 5-146258-6, Connector_PinSocket_2.54mm:PinSocket_2x06_P2.54mm_Vertical, symbol pin_header_2x12:5-146258-6
- added POWER: Screw_Terminal_01x02, symbol Connector:Screw_Terminal_01x02
- added U?: STM8S103F3M6, Package_SO:SO-20_12.8x7.5mm_P1.27mm, symbol KLIB_MCU_ST_STM8S:STM8S103F3M
Connections:
- net GND: now also CN1.GND (5), POWER.GND, U?.7 (V_{SS})
- net MISO: now also CN2.PC7 (10), U?.17 (PC7)
- net MOSI: now also CN2.PC6 (9), U?.16 (PC6)
- net RST: now also CN2.PC3 (4), U?.13 (PC3)
- net Rx: now also CN4.PD5 (10), U?.2 (PD5)
- net SCK: now also CN2.PC5 (6), U?.15 (PC5)
- net SCL: now also CN3.PB5 (5), U?.11 (PB5)
- net SDA: now also CN3.PB4 (6), U?.12 (PB4)
- net SS: now also CN2.PC4 (5), U?.14 (PC4)
- net SWIM: now also CN4.PD1 (6), U?.18 (PD1)
- net Tx: now also CN4.PD6 (11), U?.3 (PD6)
- net VDD: now also U?.9 (V_{DD})
- net ~{RST}: now also U?.4 (NRST)
- net at R_{1}.2: now also CN3.PB1 (9)
- net at R_{2}.2: now also CN3.PE7 (11)
- new net: CN1.U_{CC} (7), POWER.U_{CC} (Pin_1)
Other:
- moved on the sheet: D_{1}, D_{2}, R_{1}, R_{2}
