File: schémata/merici_stanice/merici_stanice.kicad_sch (KiCad schematic)
At the start: 17 parts, among them CN1 5-146258-6, CN2 5-146258-6, CN3 5-146258-6, CN4 5-146258-6

Commit message: changing
Parts:
- removed U?: RFID RC-522, MODULE_CEG006900, symbol CEG006900:CEG006900
- added D_{1}: GREEN, symbol Device:LED
- added D_{2}: RED, symbol Device:LED
- added R_{1}, R_{2}: 300R, symbol Device:R
- added U?: LM75A _{2}, symbol Sensor_Temperature:LM75B
- added U?: LM75A _{3}, symbol Sensor_Temperature:LM75B
- added U?: LM75A _{1}, symbol Sensor_Temperature:LM75B
Connections:
- net GND: now also D_{1}.1 (K), D_{2}.1 (K), U?.2 (GND), U?.2 (GND), U?.2 (GND)
- net MISO: no longer U?.17 (PC7)
- net MOSI: no longer U?.16 (PC6)
- net PB4: now also U?.4 (SCL), U?.4 (SCL), U?.4 (SCL)
- net PB5: now also U?.3 (SDA), U?.3 (SDA), U?.3 (SDA)
- net RST: no longer U?.13 (PC3)
- net SCK: no longer U?.15 (PC5)
- net SS: no longer U?.14 (PC4)
- net V_{DD}: now also U?.1 (+V_{CC}), U?.1 (+V_{CC}), U?.1 (+V_{CC}), U?.6 (A_{0}), U?.6 (A_{0}), U?.7 (A_{1}), U?.7 (A_{1})
- net at U?.10 (PA3): now also R_{2}.2
- net at U?.6 (PA2): now also R_{1}.2
- new net: D_{1}.2 (A), R_{1}.1
- new net: D_{2}.2 (A), R_{2}.1
Other:
- note added: "0x49"
- note added: "0x4A"
- note added: "0x4B"
- note added: "CJMCU-75"
- note removed: "Čtečka RFID karet"
- title: Security system -> Měřící stanice
- moved on the sheet: CN1, CN2, CN3, CN4, D_{1}, D_{2}, POWER, R_{1}, R_{2}
